File: 05Project/BluetoothSpeaker-5W-100W/bluetooth-speaker.kicad_pcb (KiCad board)
At the start: 2 copper layers, 16 parts, among them J1 220VAC, J2 Line-in, K1 G3MB-202P, U1 PC817, U2 MOSFET-N, U3 NE555, U4 AN6884

Commit message: Add footprint done halt
Parts:
- added D2: LED, LEDs:LED_D5.0mm_FlatTop, F.Cu at (217.8, 56.5)
- added R6: R, Resistors_SMD:R_0805_HandSoldering, F.Cu at (217.8, 41.3)
- added SW1: REV, Buttons_Switches_THT:SW_Tactile_Straight_KSA0Axx1LFTR, F.Cu at (191.1, 48.9)
- added SW2: PLAY, Buttons_Switches_THT:SW_Tactile_Straight_KSA0Axx1LFTR, F.Cu at (191.1, 30.5)
- added SW3: NEXT, Buttons_Switches_THT:SW_Tactile_Straight_KSA0Axx1LFTR, F.Cu at (191.1, 40.0)
- added U5: CSR8630-module, footprint:CSR8630-module, F.Cu at (212.7, 47.0)
- moved J1 143.6 mm to (271.8, 74.3), turned to 270 degrees
- moved K1 101.8 mm to (257.8, 69.8), turned to 270 degrees
- moved R3 88.9 mm to (241.9, 63.5), turned to 90 degrees
- moved J2 83.5 mm to (194.9, 76.8)
- moved C1 72.2 mm to (227.3, 82.5), turned to 180 degrees
- moved U2 72.0 mm to (248.3, 64.8)
- moved R2 65.2 mm to (234.3, 79.4), turned to 180 degrees
- moved U1 62.9 mm to (238.8, 76.8)
- moved R5 59.9 mm to (208.3, 67.3), turned to 180 degrees
- moved U4 53.3 mm to (183.5, 69.8)
- moved C3 47.2 mm to (203.8, 60.3)
- moved R1 45.7 mm to (189.2, 68.6), turned to 270 degrees
- moved R4 41.5 mm to (207.6, 72.4), turned to 180 degrees
- moved D1 41.2 mm to (214.0, 67.3)
- moved U3 40.6 mm to (229.2, 73.0), turned to 0 degrees
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Connections:
- K1 pad 1: Net-(K1-Pad1) -> Net-(J1-Pad1)
- K1 pad 2: Net-(K1-Pad2) -> Net-(J1-Pad2)
- K1 pad 3: Net-(K1-Pad3) -> +5V
- U2 pad 3: Net-(U2-Pad3) -> Net-(K1-Pad4)
